File: stopwater/stopwater.kicad_pcb (KiCad board)
At the start: 2 copper layers, 83.9 x 134.2 mm, 38 parts, among them J1 USB_B_Micro, J2 ~220, J3 SENS, J4 Conn_01x02_Pin, J5 Out, K1 G5LE-1, Q1 BC847, U1 TNY268P, U2 LD1117S33TR_SOT223, U4 TLP181

Commit message: added some schematics
Parts:
- removed C9: C_Polarized_Small, Capacitor_THT:C_Disc_D4.3mm_W1.9mm_P5.00mm
- removed U4: TLP181, Package_SO:SOIC-4_4.55x3.7mm_P2.54mm
- added C10: 10u, Capacitor_Tantalum_SMD:CP_EIA-3528-15_AVX-H, F.Cu at (111.1, 115.6)
- added D10: LL4148, Diode_SMD:D_MiniMELF, F.Cu at (101.6, 152.4)
- added D11: "SENS_1", LED_SMD:LED_0805_2012Metric, F.Cu at (169.5, 111.9)
- added D12: "SENS_1", LED_SMD:LED_0805_2012Metric, F.Cu at (169.5, 114.9)
- added D13: LL4148, Diode_SMD:D_MiniMELF, F.Cu at (95.2, 116.2)
- added D14: LED_Dual_AAK, LED_SMD:LED_Cree-XB, F.Cu at (169.2, 124.5)
- added D15: "SENS_3", LED_SMD:LED_0805_2012Metric, F.Cu at (169.5, 118.0)
- added D16: "SENS_4", LED_SMD:LED_0805_2012Metric, F.Cu at (169.5, 121.0)
- added D7: LL4148, Diode_SMD:D_MiniMELF, F.Cu at (113.0, 152.4)
- added D8: LL4148, Diode_SMD:D_MiniMELF, F.Cu at (109.2, 152.4)
- added D9: LL4148, Diode_SMD:D_MiniMELF, F.Cu at (105.4, 152.4)
- added J10: Conn_01x06_Socket, Connector_PinHeader_2.54mm:PinHeader_1x06_P2.54mm_Vertical, F.Cu at (118.1, 158.8)
- added J11: Conn_01x02_Socket, Connector_PinHeader_2.54mm:PinHeader_1x02_P2.54mm_Vertical, F.Cu at (162.2, 102.3)
- added J12: Out, TerminalBlock_MetzConnect:TerminalBlock_MetzConnect_Type011_RT05503HBWC_1x03_P5.00mm_Horizontal, F.Cu at (154.1, 85.4)
- added J6: Conn_01x06_Pin, Connector_PinHeader_2.54mm:PinHeader_1x06_P2.54mm_Vertical, F.Cu at (152.9, 92.7)
- added J7: Conn_01x02_Pin, Connector_PinHeader_2.54mm:PinHeader_1x02_P2.54mm_Vertical, F.Cu at (118.1, 114.9)
- added J8: Conn_01x02_Socket, Connector_PinHeader_2.54mm:PinHeader_1x02_P2.54mm_Vertical, F.Cu at (96.5, 158.8)
- added J9: Conn_01x02_Pin, Connector_PinHeader_2.54mm:PinHeader_1x02_P2.54mm_Vertical, F.Cu at (157.6, 102.3)
- added R11: 10k, Resistor_SMD:R_0603_1608Metric, F.Cu at (157.2, 111.6)
- added R12: 330, Resistor_SMD:R_0805_2012Metric, F.Cu at (204.0, 79.9)
- added R13: 680, Resistor_SMD:R_0805_2012Metric, F.Cu at (204.0, 82.9)
- added R14: 3.3k, Resistor_SMD:R_0603_1608Metric, F.Cu at (89.9, 154.3)
- added R15: 1k, Resistor_SMD:R_0603_1608Metric, F.Cu at (93.3, 148.0)
- added R16: 10k, Resistor_SMD:R_0603_1608Metric, F.Cu at (113.0, 122.3)
- added R17: 10k, Resistor_SMD:R_0603_1608Metric, F.Cu at (157.2, 114.1)
- added R18: 10k, Resistor_SMD:R_0603_1608Metric, F.Cu at (157.2, 116.7)
- added R19: 10k, Resistor_SMD:R_0603_1608Metric, F.Cu at (157.2, 119.2)
- added R20: 10k, Resistor_SMD:R_0603_1608Metric, F.Cu at (157.2, 121.7)
- added R21: 10k, Resistor_SMD:R_0603_1608Metric, F.Cu at (161.3, 111.6)
- added R22: 10k, Resistor_SMD:R_0603_1608Metric, F.Cu at (161.3, 114.1)
- added R23: 10k, Resistor_SMD:R_0603_1608Metric, F.Cu at (161.3, 116.7)
- added R24: 10k, Resistor_SMD:R_0603_1608Metric, F.Cu at (161.3, 119.2)
- added R25: 10k, Resistor_SMD:R_0603_1608Metric, F.Cu at (161.3, 121.7)
- added R26: 10k, Resistor_SMD:R_0603_1608Metric, F.Cu at (165.3, 111.6)
- added R27: 10k, Resistor_SMD:R_0603_1608Metric, F.Cu at (165.3, 114.1)
- added R28: 10k, Resistor_SMD:R_0603_1608Metric, F.Cu at (165.3, 116.7)
- added R29: 10k, Resistor_SMD:R_0603_1608Metric, F.Cu at (165.3, 119.2)
- added U3: TLP181, Package_SO:SOIC-4_4.55x3.7mm_P2.54mm, F.Cu at (202.3, 102.4)
- C3: value 0.1u -> 1u; footprint Capacitor_SMD:C_0603_1608Metric_Pad1.08x0.95mm_HandSolder -> Capacitor_SMD:C_0805_2012Metric; moved to F.Cu
- C4, D1, D2, D3, J1, Q1: moved to F.Cu
- C5: value 200u 16v -> C_Polarized_Small; footprint Capacitor_THT:CP_Radial_D8.0mm_P3.50mm -> Capacitor_THT:C_Disc_D4.3mm_W1.9mm_P5.00mm
- C7: value 100u -> 10u; footprint Capacitor_THT:CP_Radial_D5.0mm_P2.50mm -> Capacitor_Tantalum_SMD:CP_EIA-3528-15_AVX-H
- C8: value 0.1u -> 200u 16v; footprint Capacitor_SMD:C_0603_1608Metric_Pad1.08x0.95mm_HandSolder -> Capacitor_THT:CP_Radial_D8.0mm_P3.50mm
- D4: value MMSD4148 -> SS14; footprint Diode_SMD:D_SOD-123 -> Diode_SMD:D_SMA; moved to F.Cu
- D5: value SS14 -> 8v2; footprint Diode_SMD:D_SMA -> Diode_SMD:D_MiniMELF_Handsoldering; moved to F.Cu
- D6: value 8v2 -> MMSD4148; footprint Diode_SMD:D_MiniMELF_Handsoldering -> Diode_SMD:D_SOD-123; moved to F.Cu
- DD1: footprint stopwater:ESP32C3-WROOM-02 -> stopwater:ESP-WROOM-02; moved to F.Cu
- J3: value SENS -> Out; footprint TerminalBlock_MetzConnect:TerminalBlock_MetzConnect_Type011_RT05502HBWC_1x02_P5.00mm_Horizontal -> TerminalBlock_MetzConnect:TerminalBlock_MetzConnect_Type011_RT05503HBWC_1x03_P5.00mm_Horizontal
- J4: value Conn_01x02_Pin -> Conn_01x05; footprint Connector_PinSocket_2.54mm:PinSocket_1x02_P2.54mm_Vertical -> Connector_PinHeader_2.54mm:PinHeader_1x05_P2.54mm_Vertical
- R1: value 200k -> 3.3k; footprint Resistor_THT:R_Axial_DIN0411_L9.9mm_D3.6mm_P15.24mm_Horizontal -> Resistor_SMD:R_0603_1608Metric
- R10: value 330 -> 10k; footprint Resistor_SMD:R_0805_2012Metric_Pad1.20x1.40mm_HandSolder -> Resistor_SMD:R_0805_2012Metric; moved to F.Cu
- R2: value 10k -> 3.3k; footprint Resistor_SMD:R_0603_1608Metric_Pad0.98x0.95mm_HandSolder -> Resistor_SMD:R_0603_1608Metric; moved to F.Cu
- R3, R6, R8: footprint Resistor_SMD:R_0603_1608Metric_Pad0.98x0.95mm_HandSolder -> Resistor_SMD:R_0603_1608Metric; moved to F.Cu
- R4: value 1M -> 3.3k; footprint Resistor_SMD:R_1206_3216Metric_Pad1.30x1.75mm_HandSolder -> Resistor_SMD:R_0603_1608Metric; moved to F.Cu
- R5: value 1M -> 200k; footprint Resistor_SMD:R_1206_3216Metric_Pad1.30x1.75mm_HandSolder -> Resistor_THT:R_Axial_DIN0411_L9.9mm_D3.6mm_P15.24mm_Horizontal; moved to F.Cu
- R7: value 10k -> 1M; footprint Resistor_SMD:R_0805_2012Metric_Pad1.20x1.40mm_HandSolder -> Resistor_SMD:R_1206_3216Metric; moved to F.Cu
- R9: value 680 -> 1M; footprint Resistor_SMD:R_0805_2012Metric_Pad1.20x1.40mm_HandSolder -> Resistor_SMD:R_1206_3216Metric; moved to F.Cu
- moved D1 163.5 mm to (201.8, 96.5), turned to 0 degrees
- moved J2 156.8 mm to (189.2, 83.0), turned to 0 degrees
- moved F1 143.0 mm to (170.0, 101.6)
- moved R4 142.7 mm to (199.8, 84.3), turned to 0 degrees
- moved R5 138.7 mm to (187.7, 90.6), turned to 0 degrees
- moved R2 138.3 mm to (199.8, 79.3), turned to 0 degrees
- moved C4 134.8 mm to (204.2, 85.8)
- moved R7 134.2 mm to (203.8, 70.4), turned to 0 degrees
- moved U1 132.3 mm to (192.3, 54.8)
- moved K1 126.2 mm to (176.7, 79.0), turned to 0 degrees
- moved R1 120.3 mm to (199.8, 76.8)
- moved C1 119.2 mm to (189.2, 99.0), turned to 0 degrees
- moved R3 117.7 mm to (199.8, 81.8), turned to 0 degrees
- moved J5 114.4 mm to (154.1, 72.8), turned to 0 degrees
- moved R9 113.3 mm to (203.8, 73.7), turned to 0 degrees
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Connections:
- net Net-(DD1-IO18) renamed /USB_DN
- net Net-(DD1-IO19) renamed /USB_DP
- net Net-(DD1-IO4) renamed /IO_4
- C5 pad 1: +12V -> Net-(C5-plus)
- C5 pad 2: Net-(C5-minus) -> Net-(C1-plus)
- C6 pad 1: +12V -> Net-(DD1-EN)
- C8 pad 1: +3.3V -> +12V
- C8 pad 2: GND -> Net-(C5-plus)
- D4 pad 2: /REL_CTRL -> Net-(D4-A)
- D6 pad 2: Net-(D6-A) -> +12V
- DD1 pad 10: unconnected-(DD1-IO10-Pad10) -> /IO_10
- DD1 pad 11: unconnected-(DD1-RXD-Pad11) -> Net-(DD1-RXD)
- DD1 pad 12: unconnected-(DD1-TXD-Pad12) -> Net-(DD1-TXD)
- DD1 pad 15: unconnected-(DD1-IO3-Pad15) -> /IO_3
- DD1 pad 16: +3.3V -> /IO_2
- DD1 pad 17: unconnected-(DD1-IO1-Pad17) -> /IO_1
- DD1 pad 18: unconnected-(DD1-IO0-Pad18) -> /IO_0
- DD1 pad 2: +3.3V -> Net-(DD1-EN)
- DD1 pad 4: /SENSOR -> /IO_5
- DD1 pad 5: unconnected-(DD1-IO6-Pad5) -> /IO_6
- DD1 pad 6: unconnected-(DD1-IO7-Pad6) -> /IO_7
- DD1 pad 7: +3.3V -> /IO_8
- DD1 pad 8: Net-(DD1-IO9) -> /IO_9
- J1 pad 1: unconnected-(J1-VBUS-Pad1) -> Net-(D13-A)
- J3 pad 1: /SENSOR -> /power/SENSOR_1
- J4 pad 1: Net-(DD1-IO9) -> Net-(DD1-EN)
- J4 pad 2: GND -> /IO_9
- J5 pad 1: Net-(J5-Pin_1) -> /power/SENSOR_3
- J5 pad 2: Net-(J5-Pin_2) -> GND
- J5 pad 3: Net-(J5-Pin_3) -> /power/SENSOR_4
- K1 pad 1: Net-(J5-Pin_2) -> Net-(J12-Pin_2)
- K1 pad 2: /REL_CTRL -> +12V
- K1 pad 3: Net-(J5-Pin_3) -> Net-(J12-Pin_3)
- K1 pad 4: Net-(J5-Pin_1) -> Net-(J12-Pin_1)
- R1 pad 1: Net-(D2-K) -> +12V
- R1 pad 2: Net-(C1-plus) -> /power/SENSOR_1
- R10 pad 1: Net-(R10-Pad1) -> Net-(D3-K)
- R10 pad 2: Net-(D6-A) -> Net-(C4-plus)
- R2 pad 2: /SENSOR -> /power/SENSOR_2
- R3 pad 1: /SENSOR -> +12V
- R3 pad 2: GND -> /power/SENSOR_2
- R4 pad 1: Net-(R4-Pad1) -> +12V
- R4 pad 2: Net-(C1-plus) -> /power/SENSOR_4
- R5 pad 1: Net-(U1-EN/UV) -> Net-(D2-K)
- R5 pad 2: Net-(R4-Pad1) -> Net-(C1-plus)
- R7 pad 1: Net-(C4-plus) -> Net-(R7-Pad1)
- R7 pad 2: Net-(D3-K) -> Net-(C1-plus)
- R9 pad 1: GND -> Net-(U1-EN/UV)
- R9 pad 2: Net-(R10-Pad1) -> Net-(R7-Pad1)
- TR1 pad 10: Net-(C5-minus) -> Net-(C5-plus)
- TR1 pad 6: Net-(D5-A) -> Net-(D4-A)
- U2 pad 3: +12V -> /+12
Routing:
- net GND: track 0.00 -> 56.1 mm
- net +3.3V: track 0.00 -> 23.9 mm, vias 0 -> 1
- net (no net): track 0.00 -> 22.5 mm
- net /SENSOR_1: track 0.00 -> 8.85 mm
- net /SENSOR_3: track 0.00 -> 8.56 mm
- net /SENSOR_2: track 0.00 -> 6.92 mm
- net /SENSOR_4: track 0.00 -> 6.18 mm
- net Net-(DD1-EN): track 0.00 -> 4.81 mm
- added copper zone on F.Cu, net /SENSOR_1
- added copper zone on F.Cu, net /SENSOR_2
- added copper zone on F.Cu, net /SENSOR_3
- added copper zone on F.Cu, net /SENSOR_4
- added copper zone on F.Cu, net GND
Other:
- board size 83.9 x 134.2 mm -> 84 x 104.1 mm
